File: kraft80/hardware/Kraft80.kicad_sch (KiCad schematic)
At the start: 90 parts, among them CN1 +5VCC, P1 100k, SW1 SW_Push, SW2 SW_Push, SW3 SW_Push, SW4 SW_Push, SW5 SW_Push, SW6 SW_Push, SW7 SW_Push, SW8 SW_Push, U1 Z80CPU, U10 74HC04, U11 74LS273, U2 KM28C64A, U3 74LS138, U4 4093, U5 74LS273, U6 74LS245, U7 74LS32, U9 HM62256BLP, U90 HM62256BLP, U91 74LS138, U92 74LS00, U93 74LS08, U94 74LS393, U95 8251A, U96 8259A, U97 74LS32, U98 74LS393, U99 74LS74, X1 4MHz, Y1 2,4576MHz

Commit message: Update Kraft80 files.
Parts:
- added D11, D12: LED, symbol Device:LED
- added R21, R22: 1k8, symbol Device:R
Connections:
- net CPM: now also U99.5 (Q), R21.1; no longer U11.6 (Q2)
- net GNDREF: now also D11.1 (K), D12.1 (K)
- net at U99.9 (Q): now also R22.1
- new net: D11.2 (A), R21.2
- new net: D12.2 (A), R22.2
Other:
- note added: "PORTS: 00h - LEDS(W) & BUTTONS(R) 10h - LCD(W) 20h - 8251(RW) 30h - 8259A(RW) 40h - FFs(W)"
- note removed: "PORTS: 00h - LEDS(W) & BUTTONS(R) 10h - LCD(W) 20h - 8251(RW) 30h - 8259A(RW)"
- moved on the sheet: C5

Commit message: Update Kraftmon to v1.3 and schematics fixes (no build changes).
Parts:
- removed C16, C17, C8, C9, C92, C94, C95, C96: 100nF, symbol Device:C
- removed D10, D11, D12, D3, D4, D5, D6, D7, D8, D9: LED, symbol Device:LED
- removed JP1, JP2: Jumper_3_Bridged12, symbol Jumper:Jumper_3_Bridged12
- removed JP4: Jumper_2_Small_Bridged, symbol Jumper:Jumper_2_Small_Bridged
- removed LCD1: LCD16X2, Display:LCD-016N002L, symbol Display_Character:LCD-016N002L
- removed P1: 100k, symbol Device:R_Potentiometer_Trim_US
- removed R10, R11, R12, R13, R14, R15, R21, R22, R8, R9: 1k8, symbol Device:R
- removed R20: 22, symbol Device:R
- removed RP1: R_Pack08, symbol Device:R_Pack08
- removed SW1, SW2, SW3, SW4, SW5, SW6, SW7, SW8: SW_Push, symbol Switch:SW_Push
- removed U11, U5: 74LS273, symbol 74xx:74LS273
- removed unit 3 of U4
- removed unit 4 of U4
- removed U6: 74LS245, symbol 74xx:74LS245
- removed U92: 74LS00, symbol 74xx:74LS00
- removed unit 3 of U93
- removed unit 4 of U93
- removed U94, U98: 74LS393, symbol 74xx:74LS393
- removed U95: 8251A, Package_DIP:DIP-28_W15.24mm, symbol Z80Alpha:8251A
- removed U96: 8259A, Package_DIP:DIP-28_W15.24mm, symbol Interface:8259A
- removed U99: 74LS74, symbol 74xx:74LS74
- removed Y1: 2,4576MHz, Oscillator:Oscillator_DIP-14, symbol Oscillator:ACO-xxxMHz-A
- renumbered RST to RST1
Connections:
- net ~{P8251_CS}: now reaches U3.13 (O2)
- net ~{P8259_CS}: now reaches U3.12 (O3)
Other:
- added sheet kraft80-ios (kraft80-ios.kicad_sch)
- added sheet kraft80-uart-irq (kraft80-uart-irq.kicad_sch)
- note removed: "300 Hz"
- note removed: "307.2kHz 19200BPS x 16"
- moved on the sheet: C10, C13, C14, C15, C3, C5, C6, C7, C91, C97, CN1, D1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

Commit message: Lots of releases from Kraft80 scratch.
Connections:
- net ~{VID_CS}: now reaches U3.10 (O5)
Other:
- added sheet kraft80-video (kraft80-video.kicad_sch)
- note added: "PORTS: 00h - LEDS(W) & BUTTONS(R) 10h - LCD(W) 20h - 8251(RW) 30h - 8259A(RW) 40h - FFs(W) 50h - VIDEO"
- note removed: "PORTS: 00h - LEDS(W) & BUTTONS(R) 10h - LCD(W) 20h - 8251(RW) 30h - 8259A(RW) 40h - FFs(W)"
Changed lines of the file:
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@@
 	(title_block
 		(title "Kraft 80 by ARMCoder")
-		(date "2025-06-18")
+		(date "2025-07-01")
 		(rev "1.1")
 		(comment 1 "www.github.com/ARMCoderBR")
 		(comment 3 "Inspired on the project Z80 Alpha from WR Kits (www.wrkits.com.br)")
 	)
-	(text "PORTS:\n00h - LEDS(W) & BUTTONS(R)\n10h - LCD(W)\n20h - 8251(RW)\n30h - 8259A(RW)\n40h - FFs(W)"
+	(text "PORTS:\n00h - LEDS(W) & BUTTONS(R)\n10h - LCD(W)\n20h - 8251(RW)\n30h - 8259A(RW)\n40h - FFs(W)\n50h - VIDEO"
 		(exclude_from_sim no)
 		(at 249.936 148.082 0)
@@
 	(wire
 		(pts
-			(xy 257.81 124.46) (xy 261.62 124.46)
+			(xy 257.81 124.46) (xy 270.51 124.46)
 		)
 		(stroke
@@
 	(wire
 		(pts
-			(xy 270.51 123.19) (xy 261.62 123.19)
-		)
-		(stroke
-			(width 0)
-			(type default)
-		)
-	)
-	(wire
-		(pts
 			(xy 168.91 114.3) (xy 179.07 114.3)
 		)
@@
 		)
 	)
-	(wire
-		(pts
-			(xy 261.62 123.19) (xy 261.62 124.46)
-		)
-		(stroke
-			(width 0)
-			(type default)
-		)
-	)
 	(bus
 		(pts
@@
 	(wire
 		(pts
-			(xy 261.62 120.65) (xy 261.62 121.92)
-		)
-		(stroke
-			(width 0)
-			(type default)
-		)
-	)
-	(wire
-		(pts
 			(xy 151.13 49.53) (xy 167.64 49.53)
 		)
@@
 	(wire
 		(pts
-			(xy 270.51 120.65) (xy 261.62 120.65)
-		)
-		(stroke
-			(width 0)
-			(type default)
-		)
-	)
-	(wire
-		(pts
 			(xy 92.71 125.73) (xy 92.71 127)
 		)
@@
 	(wire
 		(pts
+			(xy 257.81 129.54) (xy 270.51 129.54)
+		)
+		(stroke
+			(width 0)
+			(type default)
+		)
+	)
+	(wire
+		(pts
 			(xy 151.13 62.23) (xy 167.64 62.23)
 		)
@@
 	(wire
 		(pts
-			(xy 261.62 121.92) (xy 257.81 121.92)
+			(xy 257.81 121.92) (xy 270.51 121.92)
 		)
 		(stroke
@@
 		)
 	)
-	(label "CLOCK"
-		(at 35.56 36.83 0)
-		(effects
-			(font
-				(size 1.27 1.27)
-			)
-			(justify left bottom)
-		)
-	)
 	(label "A1"
 		(at 153.67 31.75 0)
@@
 		)
 	)
-	(label "CLOCK"
-		(at 99.06 157.48 0)
-		(effects
-			(font
-				(size 1.27 1.27)
-			)
-			(justify left bottom)
-		)
-	)
 	(label "D4"
 		(at 80.01 82.55 0)
@@
 		)
 	)
+	(global_label "CLOCK"
+		(shape output)
+		(at 99.06 157.48 0)
+		(fields_autoplaced yes)
+		(effects
+			(font
+				(size 1.27 1.27)
+			)
+			(justify left)
+		)
+		(property "Intersheetrefs" "${INTERSHEET_REFS}"
+			(at 108.2138 157.48 0)
+			(effects
+				(font
+					(size 1.27 1.27)
+				)
+				(justify left)
+				(hide yes)
+			)
+		)
+	)
 	(global_label "~{INT}"
 		(shape input)
@@
 		)
 	)
+	(global_label "~{VID_CS}"
+		(shape output)
+		(at 270.51 129.54 0)
+		(fields_autoplaced yes)
+		(effects
+			(font
+				(size 1.27 1.27)
+			)
+			(justify left)
+		)
+		(property "Intersheetrefs" "${INTERSHEET_REFS}"
+			(at 279.9057 129.54 0)
+			(effects
+				(font
+					(size 1.27 1.27)
+				)
+				(justify left)
+				(hide yes)
+			)
+		)
+	)
 	(global_label "~{READ}"
 		(shape input)
@@
 	(global_label "~{P8251_CS}"
 		(shape output)
-		(at 270.51 120.65 0)
+		(at 270.51 121.92 0)
 		(fields_autoplaced yes)
 		(effects
@@
 		)
 		(property "Intersheetrefs" "${INTERSHEET_REFS}"
-			(at 283.0503 120.65 0)
+			(at 283.0503 121.92 0)
 			(effects
 				(font
@@
 	(global_label "~{P8259_CS}"
 		(shape output)
-		(at 270.51 123.19 0)
+		(at 270.51 124.46 0)
 		(fields_autoplaced yes)
 		(effects
@@
 		)
 		(property "Intersheetrefs" "${INTERSHEET_REFS}"
-			(at 283.0503 123.19 0)
+			(at 283.0503 124.46 0)
 			(effects
 				(font
@@
 		)
 	)
+	(global_label "CLOCK"
+		(shape input)
+		(at 35.56 36.83 180)
+		(fields_autoplaced yes)
+		(effects
+			(font
+				(size 1.27 1.27)
+			)
+			(justify right)
+		)
+		(property "Intersheetrefs" "${INTERSHEET_REFS}"
+			(at 26.4062 36.83 0)
+			(effects
+				(font
+					(size 1.27 1.27)
+				)
+				(justify right)
+				(hide yes)
+			)
+		)
+	)
 	(symbol
 		(lib_id "power:+5V")
@@
 				)
 			)
+		)
+	)
+	(sheet
+		(at 55.88 181.61)
+		(size 17.78 11.43)
+		(exclude_from_sim no)
+		(in_bom yes)
+		(on_board yes)
+		(dnp no)
+		(stroke
+			(width 0.1524)
+			(type solid)
+		)
+		(fill
+			(color 255 255 194 1.0000)
+		)
+		(property "Sheetname" "kraft80-video"
+			(at 57.404 184.404 0)
+			(effects
+				(font
+					(size 1.27 1.27)
+				)
+				(justify left bottom)
+			)
+		)
+		(property "Sheetfile" "kraft80-video.kicad_sch"
+			(at 55.88 202.5146 0)
+			(effects
+				(font
+					(size 1.27 1.27)
+				)
+				(justify left top)
+				(hide yes)
+			)
+		)
+		(instances
+			(project "Kraft80"
+				(path "/fd4979f9-cac6-4d50-ad9a-4fcaee298cd9"
+					(page "4")
+				)
+			)
