File: kraft80/hardware/Kraft80V2.kicad_pcb (KiCad board)
At the start: 2 copper layers, 150.6 x 171.7 mm, 139 parts, among them CN1 +5VCC, J3 Speaker, J4 Mini-DIN-6, J9 Conn_01x06_Socket, P1 100k, Q1 BC337, SW1 SW_Push, SW2 SW_Push, SW3 SW_Push, SW4 SW_Push, SW5 SW_Push, SW6 SW_Push, SW7 SW_Push, SW8 SW_Push, U1 Z84C00xxP, U10 74HC04, U11 74LS273, U12 LVL-SHFT-8CH, U13 YP-8, U15 74HC595, U16 74HC595, U17 FTDI USB ADAPTER, U18 KM28C64A, U19 TANG NANO 9K, U2 KM28C64A, U3 74LS138, U4 4093, U5 74LS273, U6 74LS245, U7 74LS32, U8 LVL-SHFT-8CH, U9 HM62256BLP, U90 HM62256BLP, U91 74LS138, U93 74LS08, U97 74LS32, U99 74LS74, X1 4MHz

Commit message: Fixes missing resistors on Kraft80 PCB.
Parts:
- added R19: 5k6, Resistor_THT:R_Axial_DIN0207_L6.3mm_D2.5mm_P2.54mm_Vertical, F.Cu at (37.9, 145.4)
- added R3: 10k, Resistor_THT:R_Axial_DIN0207_L6.3mm_D2.5mm_P2.54mm_Vertical, F.Cu at (73.3, 125.0)
- added R4: 10k, Resistor_THT:R_Axial_DIN0207_L6.3mm_D2.5mm_P2.54mm_Vertical, F.Cu at (73.3, 129.2)
- added R5: 10k, Resistor_THT:R_Axial_DIN0207_L6.3mm_D2.5mm_P2.54mm_Vertical, F.Cu at (46.8, 125.7)
- added R6: 10k, Resistor_THT:R_Axial_DIN0207_L6.3mm_D2.5mm_P2.54mm_Vertical, F.Cu at (46.8, 129.2)
Routing:
- net +5V: track 891.8 -> 945.8 mm, vias 17 -> 18
- net GNDREF: track 1658.2 -> 1663.8 mm
- net Net-(U1-~{BUSREQ}): track 0.00 -> 4.36 mm
- net ~{INT}: track 79.1 -> 82.6 mm
- net Net-(U1-~{WAIT}): track 0.00 -> 3.42 mm
- net Net-(U1-~{NMI}): track 0.00 -> 3.12 mm
Other:
- board text added: "Rev 2.0.1 ©2025 ARMCoder"
- board text removed: "Rev 2.0 ©2025 ARMCoder"

Commit message: Kraft80 PCB updates
Parts:
- moved G*** 62.3 mm to (74.1, 80.3)
- moved R39 51.4 mm to (64.3, 30.3), turned to 180 degrees
- moved J4 46.3 mm to (50.9, 29.5), turned to 90 degrees
- moved R40 46.2 mm to (64.3, 34.1), turned to 180 degrees
- moved U17 9.58 mm to (32.9, 37.7), turned to 90 degrees
- moved C2 7.90 mm to (95.9, 85.8), turned to 180 degrees
- moved RV1 7.13 mm to (64.2, 42.3), turned to 0 degrees
- moved U19 4.57 mm to (146.9, 61.7)
- moved J9 3.71 mm to (129.5, 26.4)
- moved R49 3.58 mm to (131.1, 80.7)
- moved R50 3.58 mm to (127.7, 80.7)
- moved R51 3.58 mm to (124.3, 80.7)
- moved R52 3.58 mm to (120.9, 80.7)
- moved R53 3.58 mm to (131.1, 87.8)
- moved R57 3.58 mm to (127.7, 87.7)
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Routing:
- net GNDREF: track 1663.8 -> 1526.3 mm, vias 32 -> 27
- net /kraft80V2-fpga/DISK_SCK: track 87.7 -> 113.0 mm, vias 2 -> 0
- net Net-(U19-IOB29A): track 121.7 -> 99.8 mm, vias 3 -> 2
- net /kraft80V2-fpga/CK_KBD: track 78.1 -> 99.9 mm, vias 1 -> 2
- net Net-(U17-TXD): track 172.4 -> 151.4 mm, vias 1 -> 2
- net /kraft80V2-fpga/DAT_KBD: track 57.7 -> 76.7 mm, vias 1 -> 2
- net +3V3: track 164.3 -> 182.4 mm
- net Net-(U19-IOT12B): track 46.9 -> 28.9 mm, vias 2 -> 1
- net Net-(U17-~{CTS}): track 136.2 -> 153.7 mm, vias 1 -> 2
- net Net-(U19-IOB33B): track 115.2 -> 99.4 mm, vias 3 -> 1
- net Net-(U19-IOB23B): track 106.8 -> 91.1 mm, vias 3 -> 1
- net Net-(U17-RXD): track 174.7 -> 160.1 mm
- net Net-(U12-LV3): track 58.7 -> 45.1 mm, vias 2 -> 1
- net CLOCK: track 138.0 -> 149.7 mm, vias 3 -> 4
- net Net-(U12-LV8): track 89.5 -> 80.7 mm
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Other:
- board text added: "+"
- board text added: "+5 VDC"
- board text added: "-"
- board text added: "AUX"
- board text added: "CP/M"

Commit message: Kraft80 schematic fix (audio amp) and PCB update.
Parts:
- R20: value 10k -> 2k
- R43: value 100R -> 22R
- R49, R50, R51, R52: value 10k -> 1k
- R53, R57, R58, R59: value 18k -> 1k
Connections:
- R20 pad 1: +5V -> Net-(J3-Pin_2)
Routing:
- net Net-(J3-Pin_2): track 16.8 -> 24.2 mm
- net +5V: track 946.7 -> 941.5 mm
Changed lines of the file:
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@@
 	(title_block
 		(title "Kraft80 V2.0.1")
-		(date "2025-09-30")
+		(date "2025-10-01")
 		(comment 1 "©2025 ARMCoder")
 	)
@@
 			)
 		)
-		(property "Value" "10k"
+		(property "Value" "2k"
 			(at 1.27 0.762 90)
 			(layer "F.Fab")
@@
 			(layers "*.Cu" "*.Mask")
 			(remove_unused_layers no)
-			(net 30 "+5V")
+			(net 26 "Net-(J3-Pin_2)")
 			(pintype "passive")
 		)
@@
 			)
 		)
-		(property "Value" "18k"
+		(property "Value" "1k"
 			(at 1.27 2.37 90)
 			(layer "F.Fab")
@@
 			)
 		)
-		(property "Value" "10k"
+		(property "Value" "1k"
 			(at 1.27 2.47 90)
 			(layer "F.Fab")
@@
 			)
 		)
-		(property "Value" "10k"
+		(property "Value" "1k"
 			(at 1.4832 3.0938 90)
 			(layer "F.Fab")
@@
 			)
 		)
-		(property "Value" "10k"
+		(property "Value" "1k"
 			(at 1.27 2.37 90)
 			(layer "F.Fab")
@@
 			)
 		)
-		(property "Value" "100R"
+		(property "Value" "22R"
 			(at 1.27 2.37 90)
 			(layer "F.Fab")
@@
 			)
 		)
-		(property "Value" "18k"
+		(property "Value" "1k"
 			(at 1.27 2.47 90)
 			(layer "F.Fab")
@@
 			)
 		)
-		(property "Value" "18k"
+		(property "Value" "1k"
 			(at 1.4832 3.0938 90)
 			(layer "F.Fab")
@@
 			)
 		)
-		(property "Value" "10k"
+		(property "Value" "1k"
 			(at 1.27 2.37 90)
 			(layer "F.Fab")
@@
 			)
 		)
-		(property "Value" "18k"
+		(property "Value" "1k"
 			(at 1.27 2.37 90)
 			(layer "F.Fab")
@@
 		)
 	)
+	(gr_text "+"
+		(at 79.94 40.74 0)
+		(layer "F.SilkS")
+		(effects
+			(font
+				(size 1 1)
+				(thickness 0.2)
+				(bold yes)
+			)
+			(justify left bottom)
+		)
+	)
+	(gr_text "+"
+		(at 152.78 141.91 0)
+		(layer "F.SilkS")
+		(effects
+			(font
+				(size 1 1)
+				(thickness 0.2)
+				(bold yes)
+			)
+			(justify left bottom mirror)
+		)
+	)
+	(gr_text "+"
+		(at 153.36 173.67 0)
+		(layer "F.SilkS")
+		(effects
+			(font
+				(size 1 1)
+				(thickness 0.2)
+				(bold yes)
+			)
+			(justify left bottom mirror)
+		)
+	)
 	(gr_text "+5 VDC"
 		(at 159.6 138 0)
@@
 	)
 	(segment
+		(start 79.1522 34.69)
+		(end 79.45 34.69)
+		(width 0.2)
+		(layer "F.Cu")
+		(net 26)
+	)
+	(segment
 		(start 76.8488 46.9012)
 		(end 76.8138 46.9012)
@@
 	)
 	(segment
+		(start 74.195 39.6472)
+		(end 79.1522 34.69)
+		(width 0.2)
+		(layer "F.Cu")
+		(net 26)
+	)
+	(segment
 		(start 80.85 46.73)
 		(end 80.85 36.09)
@@
 	)
 	(segment
+		(start 74.2738 39.5684)
+		(end 74.195 39.6472)
+		(width 0.2)
+		(layer "B.Cu")
+		(net 26)
+	)
+	(segment
 		(start 80.6788 46.9012)
 		(end 80.85 46.73)
@@
 	)
 	(segment
-		(start 74.2738 39.5684)
-		(end 74.195 39.6472)
-		(width 0.2)
-		(layer "B.Cu")
-		(net 30)
-	)
-	(segment
 		(start 139.51 91.74)
 		(end 132.3298 91.74)
@@
 		(layer "B.Cu")
 		(net 30)
-	)
-	(segment
-		(start 74.2738 34.5612)
-		(end 74.2738 39.5684)
-		(width 0.2)
-		(layer "B.Cu")
-		(net 30)
