File: kraft80/hardware/kraft80V2-fpga.kicad_sch (KiCad schematic)
At the start: 51 parts, among them J3 Speaker, J4 Mini-DIN-6, J9 Conn_01x06_Socket, Q1 BC337, U12 LVL-SHFT-8CH, U13 YP-8, U15 74HC595, U16 74HC595, U17 FTDI USB ADAPTER, U19 TANG NANO 9K, U8 LVL-SHFT-8CH

Commit message: Kraft80 schematic fix (audio amp) and PCB update.
Parts:
- R20: value 10k -> 2k
- R43: value 100R -> 22R
Connections:
- net +5V: no longer R20.1
- net at J3.2 (Pin_2), Q1.1 (C): now also R20.1
Changed lines of the file:
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@@
 	(title_block
 		(title "Kraft 80 V2 by ARMCoder")
-		(date "2025-09-02")
+		(date "2025-10-01")
 		(rev "2.0")
 		(comment 1 "www.github.com/ARMCoderBR")
@@
 	)
 	(junction
-		(at 261.62 66.04)
-		(diameter 0)
-		(color 0 0 0 0)
-	)
-	(junction
 		(at 194.31 123.19)
 		(diameter 0)
@@
 	)
 	(junction
+		(at 271.78 68.58)
+		(diameter 0)
+		(color 0 0 0 0)
+	)
+	(junction
 		(at 232.41 134.62)
 		(diameter 0)
@@
 	(wire
 		(pts
-			(xy 261.62 66.04) (xy 261.62 69.85)
-		)
-		(stroke
-			(width 0)
-			(type default)
-		)
-	)
-	(wire
-		(pts
 			(xy 88.9 139.7) (xy 99.06 139.7)
 		)
@@
 	(wire
 		(pts
+			(xy 261.62 68.58) (xy 271.78 68.58)
+		)
+		(stroke
+			(width 0)
+			(type default)
+		)
+	)
+	(wire
+		(pts
 			(xy 15.24 54.61) (xy 19.05 54.61)
 		)
@@
 	(wire
 		(pts
+			(xy 261.62 69.85) (xy 261.62 68.58)
+		)
+		(stroke
+			(width 0)
+			(type default)
+		)
+	)
+	(wire
+		(pts
 			(xy 93.98 95.25) (xy 93.98 100.33)
 		)
@@
 		(dnp no)
 		(property "Reference" "R20"
-			(at 262.89 70.104 0)
+			(at 263.144 72.39 0)
 			(effects
 				(font
@@
 			)
 		)
-		(property "Value" "10k"
-			(at 262.89 72.898 0)
+		(property "Value" "2k"
+			(at 263.144 74.422 0)
 			(effects
 				(font
@@
 			)
 		)
-		(property "Value" "100R"
+		(property "Value" "22R"
 			(at 270.51 64.516 0)
 			(effects
