File: AlphaPlus/Hardware/AlphaPlus.kicad_sch (KiCad schematic)
At the start: 86 parts, among them CN1 +5VCC, P1 100k, SW1 SW_Push, SW2 SW_Push, SW3 SW_Push, SW4 SW_Push, SW5 SW_Push, SW6 SW_Push, SW7 SW_Push, SW8 SW_Push, U1 Z80CPU, U10 74HC04, U11 74LS273, U2 KM28C64A, U3 74LS138, U4 4093, U5 74LS273, U6 74LS245, U7 74LS02, U8 74LS08, U9 HM62256BLP, U90 HM62256BLP, U91 74LS138, U92 74LS00, U93 74LS08, X1 4MHz

Commit message: Updates.
Parts:
- removed C92: 100nF, symbol Device:C
- removed U92: 74LS00, symbol 74xx:74LS00
Connections:
- net ~{IOEN} is gone; now on net ~{IORQ}: U7.2, U7.8
Other:
- moved on the sheet: C10, C11

Commit message: Created Z80 Alpha and Alpha Plus PCB; Fixes missing resistors on Kraft80 PCB.
Parts:
- removed RP1: R_Pack08, symbol Device:R_Pack08
- removed U1: Z80CPU, symbol CPU:Z80CPU
- added RN1: R_Network08, Resistor_THT:R_Array_SIP9, symbol Device:R_Network08
- added U1: Z84C00xxP, Package_DIP:DIP-40_W15.24mm, symbol CPU:Z84C00xxP
- added unit 7 of U10
- added unit 5 of U4
- added unit 5 of U7
- added unit 5 of U8
- added unit 5 of U93
- renumbered RST to RST1
Connections:
- net +5V: now also RN1.1 (common), U1.11 (V_{CC}), U10.14 (VCC), U4.14 (VCC), U7.14 (VCC), U8.14 (VCC), U93.14 (VCC)
- net A0: now also U1.30 (A_{0})
- net A1: now also U1.31 (A_{1})
- net A10: now also U1.40 (A_{10})
- net A11: now also U1.1 (A_{11})
- net A12: now also U1.2 (A_{12})
- net A13: now also U1.3 (A_{13})
- net A14: now also U1.4 (A_{14})
- net A15: now also U1.5 (A_{15})
- net A2: now also U1.32 (A_{2})
- net A3: now also U1.33 (A_{3})
- net A4: now also U1.34 (A_{4})
- net A5: now also U1.35 (A_{5})
- net A6: now also U1.36 (A_{6})
- net A7: now also U1.37 (A_{7})
- net A8: now also U1.38 (A_{8})
- net A9: now also U1.39 (A_{9})
- net CLOCK: now also U1.6 (CLK)
- net D0: now also U1.14 (D_{0})
- net D1: now also U1.15 (D_{1})
- net D2: now also U1.12 (D_{2})
- net D3: now also U1.8 (D_{3})
- net D4: now also U1.7 (D_{4})
- net D5: now also U1.9 (D_{5})
- net D6: now also U1.10 (D_{6})
- net D7: now also U1.13 (D_{7})
- net GNDREF: now also U1.29 (GND), U10.7 (GND), U4.7 (GND), U7.7 (GND), U8.7 (GND), U93.7 (GND)
- net PX0: now also RN1.2 (R1)
- net PX1: now also RN1.3 (R2)
- net PX2: now also RN1.4 (R3)
- net PX3: now also RN1.5 (R4)
- net PX4: now also RN1.6 (R5)
- net PX5: now also RN1.7 (R6)
- net PX6: now also RN1.8 (R7)
- net PX7: now also RN1.9 (R8)
- net ~{INT}: now also U1.16 (~{INT})
- net ~{IORQ}: now also U1.20 (~{IORQ})
- net ~{MREQ}: now also U1.19 (~{MREQ})
- net ~{READ}: now also U1.21 (~{RD})
- net ~{RESET}: now also U1.26 (~{RESET})
- net ~{WRITE}: now also U1.22 (~{WR})
- net at R6.2: now also U1.17 (~{NMI})
- net at R3.2: now also U1.25 (~{BUSREQ})
- net at R4.2: now also U1.24 (~{WAIT})
Other:
- note added: "GND"
- moved on the sheet: R3, R4, R5, R6
