File: AlphaPlus/Hardware/AlphaPlus.kicad_pcb (KiCad board)
At the start: 2 copper layers, 150.6 x 110.4 mm, 88 parts, among them CN1 +5VCC, P1 100k, SW1 SW_Push, SW2 SW_Push, SW3 SW_Push, SW4 SW_Push, SW5 SW_Push, SW6 SW_Push, SW7 SW_Push, SW8 SW_Push, U1 Z84C00xxP, U10 74HC04, U11 74LS273, U2 KM28C64A, U3 74LS138, U4 4093, U5 74LS273, U6 74LS245, U7 74LS02, U8 74LS08, U9 HM62256BLP, U90 HM62256BLP, U91 74LS138, U93 74LS08, X1 4MHz

Commit message: Sysmon updates. AlphaPlus PCB update.
Parts:
- moved C7 2.06 mm to (157.9, 139.1)
- moved C6 2.06 mm to (153.3, 139.1)
- moved R7 1.99 mm to (165.6, 147.7)
- moved D2 1.89 mm to (158.1, 147.7)
Routing:
- net GNDREF: track 985.7 -> 982.1 mm
- net /D3: track 221.4 -> 222.4 mm
- net Net-(U1-~{BUSREQ}): track 66.7 -> 66.0 mm
- net Net-(U10-Pad11): track 86.8 -> 86.2 mm
- net /PORTB: track 57.9 -> 57.4 mm
Other:
- board text added: "+"
- board text added: "+5 VDC"
- board text added: "-"
